File: hardware/cba/kaman/io_port.kicad_sch (KiCad schematic)
At the start: 12 parts, among them J1 Conn_01x04_Pin, J2 Conn_01x04_Pin, J4 USB_C_Receptacle_USB2.0_16P, U6 CH340C, U7 PRTR5V0U2D

Commit message: hw(pcb): unorganized overlay 0.1v pcb
Parts:
- removed C10: 100nF, Capacitor_SMD:C_0402_1005Metric_Pad0.74x0.62mm_HandSolder, symbol Device:C
- added TP1: TestPoint, Connector_Pin:Pin_D1.0mm_L10.0mm, symbol Connector:TestPoint
Connections:
- net USB2_N: now reaches U6.5 (UD+), U7.1 (I/O1)
- net USB2_P: now reaches U6.6 (UD-), U7.3 (I/O2)
- net USB_P: now reaches J4.A6 (D+), J4.B6 (D+), U7.4 (I/O2)
- net USB_N: now reaches J4.A7 (D-), J4.B7 (D-), U7.6 (I/O1)
- no-connect marks 7 -> 8
Changed lines of the file:
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@@
 	)
 	(junction
-		(at 73.66 33.02)
-		(diameter 0)
-		(color 0 0 0 0)
-	)
-	(junction
 		(at 55.88 25.4)
 		(diameter 0)
@@
 		(at 31.75 45.72)
 	)
+	(no_connect
+		(at 68.58 71.12)
+	)
 	(wire
 		(pts
@@
 	(wire
 		(pts
-			(xy 52.07 38.1) (xy 68.58 38.1)
-		)
-		(stroke
-			(width 0)
-			(type default)
-		)
-	)
-	(wire
-		(pts
 			(xy 81.28 30.48) (xy 81.28 29.21)
 		)
@@
 	(wire
 		(pts
-			(xy 52.07 40.64) (xy 68.58 40.64)
+			(xy 92.71 27.94) (xy 93.98 27.94)
 		)
 		(stroke
@@
 	(wire
 		(pts
-			(xy 92.71 27.94) (xy 93.98 27.94)
+			(xy 25.4 48.26) (xy 31.75 48.26)
 		)
 		(stroke
@@
 	(wire
 		(pts
-			(xy 25.4 48.26) (xy 31.75 48.26)
+			(xy 20.32 86.36) (xy 29.21 86.36)
 		)
 		(stroke
@@
 	(wire
 		(pts
-			(xy 20.32 86.36) (xy 29.21 86.36)
+			(xy 52.07 38.1) (xy 68.58 38.1)
 		)
 		(stroke
@@
 	(wire
 		(pts
-			(xy 21.59 82.55) (xy 21.59 83.82)
+			(xy 78.74 38.1) (xy 93.98 38.1)
 		)
 		(stroke
@@
 	(wire
 		(pts
-			(xy 92.71 30.48) (xy 93.98 30.48)
+			(xy 21.59 82.55) (xy 21.59 83.82)
 		)
 		(stroke
@@
 	(wire
 		(pts
-			(xy 85.09 30.48) (xy 81.28 30.48)
+			(xy 92.71 30.48) (xy 93.98 30.48)
 		)
 		(stroke
@@
 	(wire
 		(pts
-			(xy 85.09 27.94) (xy 81.28 27.94)
+			(xy 85.09 30.48) (xy 81.28 30.48)
 		)
 		(stroke
@@
 	(wire
 		(pts
-			(xy 72.39 33.02) (xy 73.66 33.02)
+			(xy 85.09 27.94) (xy 81.28 27.94)
 		)
 		(stroke
@@
 	(wire
 		(pts
-			(xy 78.74 38.1) (xy 93.98 38.1)
+			(xy 20.32 83.82) (xy 21.59 83.82)
 		)
 		(stroke
@@
 	(wire
 		(pts
-			(xy 20.32 83.82) (xy 21.59 83.82)
+			(xy 92.71 22.86) (xy 93.98 22.86)
 		)
 		(stroke
@@
 	(wire
 		(pts
-			(xy 92.71 22.86) (xy 93.98 22.86)
+			(xy 52.07 40.64) (xy 68.58 40.64)
 		)
 		(stroke
@@
 		)
 	)
+	(label "USB_N"
+		(at 80.01 38.1 0)
+		(effects
+			(font
+				(size 1.27 1.27)
+			)
+			(justify left bottom)
+		)
+	)
+	(label "USB2_P"
+		(at 54.61 40.64 0)
+		(effects
+			(font
+				(size 1.27 1.27)
+			)
+			(justify left bottom)
+		)
+	)
+	(label "USB2_N"
+		(at 54.61 38.1 0)
+		(effects
+			(font
+				(size 1.27 1.27)
+			)
+			(justify left bottom)
+		)
+	)
+	(label "USB_P"
+		(at 80.01 40.64 0)
+		(effects
+			(font
+				(size 1.27 1.27)
+			)
+			(justify left bottom)
+		)
+	)
 	(global_label "SDA Oled"
 		(shape bidirectional)
@@
 		)
 	)
-	(netclass_flag ""
-		(length 2.54)
-		(shape round)
-		(at 82.55 40.64 180)
-		(fields_autoplaced yes)
-		(effects
-			(font
-				(size 1.27 1.27)
-			)
-			(justify right bottom)
-		)
-		(property "Netclass" "USB Diff"
-			(at 83.2485 43.18 0)
-			(show_name no)
-			(do_not_autoplace no)
-			(effects
-				(font
-					(size 1.27 1.27)
-				)
-				(justify left)
-			)
-		)
-		(property "Component Class" ""
-			(at -109.22 107.95 0)
-			(show_name no)
-			(do_not_autoplace no)
-			(effects
-				(font
-					(size 1.27 1.27)
-					(italic yes)
-				)
-				(justify right)
-			)
-		)
-	)
-	(netclass_flag ""
-		(length 2.54)
-		(shape round)
-		(at 53.34 38.1 0)
-		(fields_autoplaced yes)
-		(effects
-			(font
-				(size 1.27 1.27)
-			)
-			(justify left bottom)
-		)
-		(property "Netclass" "USB Diff"
-			(at 54.0385 35.56 0)
-			(show_name no)
-			(do_not_autoplace no)
-			(effects
-				(font
-					(size 1.27 1.27)
-				)
-				(justify left)
-			)
-		)
-		(property "Component Class" ""
-			(at -138.43 -29.21 0)
-			(show_name no)
-			(do_not_autoplace no)
-			(effects
-				(font
-					(size 1.27 1.27)
-					(italic yes)
-				)
-			)
-		)
-	)
-	(netclass_flag ""
-		(length 2.54)
-		(shape round)
-		(at 53.34 40.64 180)
-		(fields_autoplaced yes)
-		(effects
-			(font
-				(size 1.27 1.27)
-			)
-			(justify right bottom)
-		)
-		(property "Netclass" "USB Diff"
-			(at 54.0385 43.18 0)
-			(show_name no)
-			(do_not_autoplace no)
-			(effects
-				(font
-					(size 1.27 1.27)
-				)
-				(justify left)
-			)
-		)
-		(property "Component Class" ""
-			(at -138.43 107.95 0)
-			(show_name no)
-			(do_not_autoplace no)
-			(effects
-				(font
-					(size 1.27 1.27)
-					(italic yes)
-				)
-				(justify right)
-			)
-		)
-	)
-	(netclass_flag ""
-		(length 2.54)
-		(shape round)
-		(at 82.55 38.1 0)
-		(fields_autoplaced yes)
-		(effects
-			(font
-				(size 1.27 1.27)
-			)
-			(justify left bottom)
-		)
-		(property "Netclass" "USB Diff"
-			(at 83.2485 35.56 0)
-			(show_name no)
-			(do_not_autoplace no)
-			(effects
-				(font
-					(size 1.27 1.27)
-				)
-				(justify left)
-			)
-		)
-		(property "Component Class" ""
-			(at -109.22 -29.21 0)
-			(show_name no)
-			(do_not_autoplace no)
-			(effects
-				(font
-					(size 1.27 1.27)
-					(italic yes)
-				)
-			)
-		)
-	)
 	(symbol
 		(lib_id "power:+3.3V")
@@
 	)
 	(symbol
-		(lib_id "Device:C")
-		(at 68.58 33.02 90)
-		(unit 1)
-		(body_style 1)
-		(exclude_from_sim no)
-		(in_bom yes)
-		(on_board yes)
-		(in_pos_files yes)
-		(dnp no)
-		(property "Reference" "C10"
-			(at 66.802 27.432 90)
-			(show_name no)
-			(do_not_autoplace no)
-			(effects
-				(font
-					(size 1.27 1.27)
-				)
-			)
-		)
-		(property "Value" "100nF"
-			(at 68.072 29.464 90)
-			(show_name no)
-			(do_not_autoplace no)
-			(effects
-				(font
-					(size 1.27 1.27)
-				)
-			)
-		)
-		(property "Footprint" "Capacitor_SMD:C_0402_1005Metric_Pad0.74x0.62mm_HandSolder"
-			(at 72.39 32.0548 0)
-			(hide yes)
-			(show_name no)
-			(do_not_autoplace no)
-			(effects
-				(font
-					(size 1.27 1.27)
-				)
-			)
-		)
-		(property "Datasheet" ""
-			(at 68.58 33.02 0)
-			(hide yes)
-			(show_name no)
-			(do_not_autoplace no)
-			(effects
-				(font
-					(size 1.27 1.27)
-				)
-			)
-		)
-		(property "Description" "Unpolarized capacitor"
-			(at 68.58 33.02 0)
-			(hide yes)
-			(show_name no)
-			(do_not_autoplace no)
-			(effects
-				(font
-					(size 1.27 1.27)
-				)
-			)
-		)
-		(pin "1"
-		)
-		(pin "2"
-		)
-		(instances
-			(project "Template"
-				(path "/b7abe575-2b7a-4e47-9046-9769d7102f9d/c3e404eb-2e1f-4ab9-8da3-bc1a9ff0af28/5567a483-a138-4241-99fb-eb385b2c8ebc"
-					(reference "C10")
-					(unit 1)
-				)
-			)
-		)
-	)
-	(symbol
 		(lib_id "power:+3.3V")
 		(at 25.4 74.93 0)
@@
 	)
 	(symbol
-		(lib_id "power:GND")
-		(at 64.77 33.02 0)
+		(lib_id "Connector:TestPoint")
+		(at 93.98 115.57 0)
 		(unit 1)
 		(body_style 1)
@@
 		(dnp no)
 		(fields_autoplaced yes)
-		(property "Reference" "#PWR026"
-			(at 64.77 39.37 0)
-			(hide yes)
+		(property "Reference" "TP1"
+			(at 96.52 110.9979 0)
 			(show_name no)
 			(do_not_autoplace no)
@@
 					(size 1.27 1.27)
 				)
+				(justify left)
 			)
 		)
-		(property "Value" "GND"
-			(at 64.7699 36.83 90)
-			(hide yes)
+		(property "Value" "TestPoint"
+			(at 96.52 113.5379 0)
 			(show_name no)
 			(do_not_autoplace no)
@@
 					(size 1.27 1.27)
 				)
-				(justify right)
+				(justify left)
 			)
 		)
-		(property "Footprint" ""
-			(at 64.77 33.02 0)
+		(property "Footprint" "Connector_Pin:Pin_D1.0mm_L10.0mm"
+			(at 99.06 115.57 0)
 			(hide yes)
 			(show_name no)
@@
 		)
 		(property "Datasheet" ""
-			(at 64.77 33.02 0)
+			(at 99.06 115.57 0)
 			(hide yes)
 			(show_name no)
@@
 			)
 		)
-		(property "Description" "Power symbol creates a global label with name \"GND\" , ground"
-			(at 64.77 33.02 0)
+		(property "Description" "test point"
+			(at 93.98 115.57 0)
 			(hide yes)
 			(show_name no)
@@
 			(project "Template"
 				(path "/b7abe575-2b7a-4e47-9046-9769d7102f9d/c3e404eb-2e1f-4ab9-8da3-bc1a9ff0af28/5567a483-a138-4241-99fb-eb385b2c8ebc"
-					(reference "#PWR026")
+					(reference "TP1")
 					(unit 1)
 				)
