File: hardware/cba/kaman/io_port.kicad_sch (KiCad schematic)
At the start: 12 parts, among them J1 Conn_01x04_Pin, J2 Conn_01x04_Pin, J4 USB_C_Receptacle_USB2.0_16P, U6 CH340C, U7 PRTR5V0U2D

Commit message: hw(schematic): add a power switch for 3.3v
To turn off the board with the input power still connected a dip switch
with a power switch has been added and it will take care of currnet
limiting to 1A and reverse currents
Parts:
- removed TP1: TestPoint, Connector_Pin:Pin_D1.0mm_L10.0mm, symbol Connector:TestPoint
Changed lines of the file:
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@@
-	)
-	(symbol
-		(lib_id "Connector:TestPoint")
-		(at 93.98 115.57 0)
-		(unit 1)
-		(body_style 1)
-		(exclude_from_sim no)
-		(in_bom yes)
-		(on_board yes)
-		(in_pos_files yes)
-		(dnp no)
-		(fields_autoplaced yes)
-		(property "Reference" "TP1"
-			(at 96.52 110.9979 0)
-			(show_name no)
-			(do_not_autoplace no)
-			(effects
-				(font
-					(size 1.27 1.27)
-				)
-				(justify left)
-			)
-		)
-		(property "Value" "TestPoint"
-			(at 96.52 113.5379 0)
-			(show_name no)
-			(do_not_autoplace no)
-			(effects
-				(font
-					(size 1.27 1.27)
-				)
-				(justify left)
-			)
-		)
-		(property "Footprint" "Connector_Pin:Pin_D1.0mm_L10.0mm"
-			(at 99.06 115.57 0)
-			(hide yes)
-			(show_name no)
-			(do_not_autoplace no)
-			(effects
-				(font
-					(size 1.27 1.27)
-				)
-			)
-		)
-		(property "Datasheet" ""
-			(at 99.06 115.57 0)
-			(hide yes)
-			(show_name no)
-			(do_not_autoplace no)
-			(effects
-				(font
-					(size 1.27 1.27)
-				)
-			)
-		)
-		(property "Description" "test point"
-			(at 93.98 115.57 0)
-			(hide yes)
-			(show_name no)
-			(do_not_autoplace no)
-			(effects
-				(font
-					(size 1.27 1.27)
-				)
-			)
-		)
-		(pin "1"
-		)
-		(instances
-			(project "Template"
-				(path "/b7abe575-2b7a-4e47-9046-9769d7102f9d/c3e404eb-2e1f-4ab9-8da3-bc1a9ff0af28/5567a483-a138-4241-99fb-eb385b2c8ebc"
-					(reference "TP1")
-					(unit 1)
-				)
-			)
-		)
 	)
 	(symbol

Commit message: hw(schematic): fix the wrong usb connection
Connections:
- net USB2_N: now also U6.6 (UD-), U7.3 (I/O2); no longer U6.5 (UD+), U7.1 (I/O1)
- net USB2_P: now also U6.5 (UD+), U7.1 (I/O1); no longer U6.6 (UD-), U7.3 (I/O2)
- net USB_N: now also U7.4 (I/O2); no longer U7.6 (I/O1)
- net USB_P: now also U7.6 (I/O1); no longer U7.4 (I/O2)
Changed lines of the file:
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@@
 	(wire
 		(pts
+			(xy 82.55 40.64) (xy 85.09 38.1)
+		)
+		(stroke
+			(width 0)
+			(type default)
+		)
+	)
+	(wire
+		(pts
+			(xy 82.55 38.1) (xy 78.74 38.1)
+		)
+		(stroke
+			(width 0)
+			(type default)
+		)
+	)
+	(wire
+		(pts
 			(xy 92.71 27.94) (xy 93.98 27.94)
 		)
@@
 	(wire
 		(pts
+			(xy 85.09 38.1) (xy 93.98 38.1)
+		)
+		(stroke
+			(width 0)
+			(type default)
+		)
+	)
+	(wire
+		(pts
 			(xy 93.98 35.56) (xy 93.98 38.1)
 		)
@@
 	(wire
 		(pts
+			(xy 78.74 40.64) (xy 82.55 40.64)
+		)
+		(stroke
+			(width 0)
+			(type default)
+		)
+	)
+	(wire
+		(pts
 			(xy 20.32 88.9) (xy 31.75 88.9)
 		)
@@
 	(wire
 		(pts
-			(xy 78.74 38.1) (xy 93.98 38.1)
+			(xy 21.59 82.55) (xy 21.59 83.82)
 		)
 		(stroke
@@
 	(wire
 		(pts
-			(xy 21.59 82.55) (xy 21.59 83.82)
+			(xy 85.09 40.64) (xy 93.98 40.64)
 		)
 		(stroke
@@
 	(wire
 		(pts
-			(xy 52.07 40.64) (xy 68.58 40.64)
+			(xy 85.09 40.64) (xy 82.55 38.1)
 		)
 		(stroke
@@
 	(wire
 		(pts
-			(xy 25.4 33.02) (xy 31.75 33.02)
+			(xy 52.07 40.64) (xy 68.58 40.64)
 		)
 		(stroke
@@
 	(wire
 		(pts
-			(xy 78.74 40.64) (xy 93.98 40.64)
+			(xy 25.4 33.02) (xy 31.75 33.02)
 		)
 		(stroke
@@
 		)
 	)
-	(label "USB_N"
-		(at 80.01 38.1 0)
+	(label "USB2_P"
+		(at 57.15 38.1 0)
 		(effects
 			(font
@@
 		)
 	)
-	(label "USB2_P"
-		(at 54.61 40.64 0)
+	(label "USB_N"
+		(at 86.36 38.1 0)
 		(effects
 			(font
@@
 		)
 	)
-	(label "USB2_N"
-		(at 54.61 38.1 0)
+	(label "USB_P"
+		(at 86.36 40.64 0)
 		(effects
 			(font
@@
 		)
 	)
-	(label "USB_P"
-		(at 80.01 40.64 0)
+	(label "USB2_N"
+		(at 57.15 40.64 0)
 		(effects
 			(font
@@
 		)
 		(instances
+			(project "io_port"
+				(path "/663f614b-864a-4628-a976-924725dd2a5c"
+					(reference "#PWR034")
+					(unit 1)
+				)
+			)
 			(project "Template"
 				(path "/b7abe575-2b7a-4e47-9046-9769d7102f9d/c3e404eb-2e1f-4ab9-8da3-bc1a9ff0af28/5567a483-a138-4241-99fb-eb385b2c8ebc"
@@
 		)
 		(instances
+			(project "io_port"
+				(path "/663f614b-864a-4628-a976-924725dd2a5c"
+					(reference "#PWR029")
+					(unit 1)
+				)
+			)
 			(project "Template"
 				(path "/b7abe575-2b7a-4e47-9046-9769d7102f9d/c3e404eb-2e1f-4ab9-8da3-bc1a9ff0af28/5567a483-a138-4241-99fb-eb385b2c8ebc"
@@
 		)
 		(instances
+			(project "io_port"
+				(path "/663f614b-864a-4628-a976-924725dd2a5c"
+					(reference "C13")
+					(unit 1)
+				)
+			)
 			(project "Template"
 				(path "/b7abe575-2b7a-4e47-9046-9769d7102f9d/c3e404eb-2e1f-4ab9-8da3-bc1a9ff0af28/5567a483-a138-4241-99fb-eb385b2c8ebc"
@@
 		)
 		(instances
+			(project "io_port"
+				(path "/663f614b-864a-4628-a976-924725dd2a5c"
+					(reference "R11")
+					(unit 1)
+				)
+			)
 			(project "Template"
 				(path "/b7abe575-2b7a-4e47-9046-9769d7102f9d/c3e404eb-2e1f-4ab9-8da3-bc1a9ff0af28/5567a483-a138-4241-99fb-eb385b2c8ebc"
@@
 		)
 		(instances
+			(project "io_port"
+				(path "/663f614b-864a-4628-a976-924725dd2a5c"
+					(reference "#PWR046")
+					(unit 1)
+				)
+			)
 			(project "Template"
 				(path "/b7abe575-2b7a-4e47-9046-9769d7102f9d/c3e404eb-2e1f-4ab9-8da3-bc1a9ff0af28/5567a483-a138-4241-99fb-eb385b2c8ebc"
@@
 		)
 		(instances
+			(project "io_port"
+				(path "/663f614b-864a-4628-a976-924725dd2a5c"
+					(reference "R10")
+					(unit 1)
+				)
+			)
 			(project "Template"
 				(path "/b7abe575-2b7a-4e47-9046-9769d7102f9d/c3e404eb-2e1f-4ab9-8da3-bc1a9ff0af28/5567a483-a138-4241-99fb-eb385b2c8ebc"
@@
 		)
 		(instances
+			(project "io_port"
+				(path "/663f614b-864a-4628-a976-924725dd2a5c"
+					(reference "R13")
+					(unit 1)
+				)
+			)
 			(project "Template"
 				(path "/b7abe575-2b7a-4e47-9046-9769d7102f9d/c3e404eb-2e1f-4ab9-8da3-bc1a9ff0af28/5567a483-a138-4241-99fb-eb385b2c8ebc"
@@
 		)
 		(instances
+			(project "io_port"
+				(path "/663f614b-864a-4628-a976-924725dd2a5c"
+					(reference "#PWR031")
+					(unit 1)
+				)
+			)
 			(project "Template"
 				(path "/b7abe575-2b7a-4e47-9046-9769d7102f9d/c3e404eb-2e1f-4ab9-8da3-bc1a9ff0af28/5567a483-a138-4241-99fb-eb385b2c8ebc"
@@
 		)
 		(instances
+			(project "io_port"
+				(path "/663f614b-864a-4628-a976-924725dd2a5c"
+					(reference "#PWR028")
+					(unit 1)
+				)
+			)
 			(project "Template"
 				(path "/b7abe575-2b7a-4e47-9046-9769d7102f9d/c3e404eb-2e1f-4ab9-8da3-bc1a9ff0af28/5567a483-a138-4241-99fb-eb385b2c8ebc"
@@
 		)
 		(instances
+			(project "io_port"
+				(path "/663f614b-864a-4628-a976-924725dd2a5c"
+					(reference "#PWR033")
+					(unit 1)
+				)
+			)
 			(project "Template"
 				(path "/b7abe575-2b7a-4e47-9046-9769d7102f9d/c3e404eb-2e1f-4ab9-8da3-bc1a9ff0af28/5567a483-a138-4241-99fb-eb385b2c8ebc"
@@
 		)
 		(instances
+			(project "io_port"
+				(path "/663f614b-864a-4628-a976-924725dd2a5c"
+					(reference "D7")
+					(unit 1)
+				)
+			)
 			(project "Template"
 				(path "/b7abe575-2b7a-4e47-9046-9769d7102f9d/c3e404eb-2e1f-4ab9-8da3-bc1a9ff0af28/5567a483-a138-4241-99fb-eb385b2c8ebc"
@@
 		)
 		(instances
+			(project "io_port"
+				(path "/663f614b-864a-4628-a976-924725dd2a5c"
+					(reference "#PWR038")
+					(unit 1)
+				)
+			)
 			(project "Template"
 				(path "/b7abe575-2b7a-4e47-9046-9769d7102f9d/c3e404eb-2e1f-4ab9-8da3-bc1a9ff0af28/5567a483-a138-4241-99fb-eb385b2c8ebc"
@@
 		)
 		(instances
+			(project "io_port"
+				(path "/663f614b-864a-4628-a976-924725dd2a5c"
+					(reference "U7")
+					(unit 1)
+				)
+			)
 			(project "Template"
 				(path "/b7abe575-2b7a-4e47-9046-9769d7102f9d/c3e404eb-2e1f-4ab9-8da3-bc1a9ff0af28/5567a483-a138-4241-99fb-eb385b2c8ebc"
@@
 		)
 		(instances
+			(project "io_port"
+				(path "/663f614b-864a-4628-a976-924725dd2a5c"
+					(reference "J1")
+					(unit 1)
+				)
+			)
 			(project "Template"
 				(path "/b7abe575-2b7a-4e47-9046-9769d7102f9d/c3e404eb-2e1f-4ab9-8da3-bc1a9ff0af28/5567a483-a138-4241-99fb-eb385b2c8ebc"
@@
 		)
 		(instances
+			(project "io_port"
+				(path "/663f614b-864a-4628-a976-924725dd2a5c"
+					(reference "J4")
+					(unit 1)
+				)
+			)
 			(project "Template"
 				(path "/b7abe575-2b7a-4e47-9046-9769d7102f9d/c3e404eb-2e1f-4ab9-8da3-bc1a9ff0af28/5567a483-a138-4241-99fb-eb385b2c8ebc"
@@
 		)
 		(instances
+			(project "io_port"
+				(path "/663f614b-864a-4628-a976-924725dd2a5c"
+					(reference "#PWR024")
+					(unit 1)
+				)
+			)
 			(project "Template"
 				(path "/b7abe575-2b7a-4e47-9046-9769d7102f9d/c3e404eb-2e1f-4ab9-8da3-bc1a9ff0af28/5567a483-a138-4241-99fb-eb385b2c8ebc"
@@
 		)
 		(instances
+			(project "io_port"
+				(path "/663f614b-864a-4628-a976-924725dd2a5c"
+					(reference "#PWR032")
+					(unit 1)
+				)
+			)
 			(project "Template"
 				(path "/b7abe575-2b7a-4e47-9046-9769d7102f9d/c3e404eb-2e1f-4ab9-8da3-bc1a9ff0af28/5567a483-a138-4241-99fb-eb385b2c8ebc"
@@
 		)
 		(instances
+			(project "io_port"
+				(path "/663f614b-864a-4628-a976-924725dd2a5c"
+					(reference "#PWR025")
+					(unit 1)
+				)
+			)
 			(project "Template"
 				(path "/b7abe575-2b7a-4e47-9046-9769d7102f9d/c3e404eb-2e1f-4ab9-8da3-bc1a9ff0af28/5567a483-a138-4241-99fb-eb385b2c8ebc"
@@
 		)
 		(instances
+			(project "io_port"
+				(path "/663f614b-864a-4628-a976-924725dd2a5c"
+					(reference "#PWR027")
+					(unit 1)
+				)
+			)
 			(project "Template"
 				(path "/b7abe575-2b7a-4e47-9046-9769d7102f9d/c3e404eb-2e1f-4ab9-8da3-bc1a9ff0af28/5567a483-a138-4241-99fb-eb385b2c8ebc"
@@
 		)
 		(instances
+			(project "io_port"
+				(path "/663f614b-864a-4628-a976-924725dd2a5c"
+					(reference "R12")
+					(unit 1)
+				)
+			)
 			(project "Template"
 				(path "/b7abe575-2b7a-4e47-9046-9769d7102f9d/c3e404eb-2e1f-4ab9-8da3-bc1a9ff0af28/5567a483-a138-4241-99fb-eb385b2c8ebc"
@@
 		)
 		(instances
+			(project "io_port"
+				(path "/663f614b-864a-4628-a976-924725dd2a5c"
+					(reference "#PWR036")
+					(unit 1)
+				)
+			)
 			(project "Template"
 				(path "/b7abe575-2b7a-4e47-9046-9769d7102f9d/c3e404eb-2e1f-4ab9-8da3-bc1a9ff0af28/5567a483-a138-4241-99fb-eb385b2c8ebc"
@@
 		)
 		(instances
+			(project "io_port"
+				(path "/663f614b-864a-4628-a976-924725dd2a5c"
+					(reference "#PWR035")
+					(unit 1)
+				)
+			)
 			(project "Template"
 				(path "/b7abe575-2b7a-4e47-9046-9769d7102f9d/c3e404eb-2e1f-4ab9-8da3-bc1a9ff0af28/5567a483-a138-4241-99fb-eb385b2c8ebc"
@@
 		)
 		(instances
+			(project "io_port"
+				(path "/663f614b-864a-4628-a976-924725dd2a5c"
+					(reference "U6")
+					(unit 1)
+				)
+			)
 			(project "Template"
 				(path "/b7abe575-2b7a-4e47-9046-9769d7102f9d/c3e404eb-2e1f-4ab9-8da3-bc1a9ff0af28/5567a483-a138-4241-99fb-eb385b2c8ebc"
@@
 		)
 		(instances
+			(project "io_port"
+				(path "/663f614b-864a-4628-a976-924725dd2a5c"
+					(reference "J2")
+					(unit 1)
+				)
+			)
 			(project "Template"
 				(path "/b7abe575-2b7a-4e47-9046-9769d7102f9d/c3e404eb-2e1f-4ab9-8da3-bc1a9ff0af28/5567a483-a138-4241-99fb-eb385b2c8ebc"
@@
 		)
 		(instances
+			(project "io_port"
+				(path "/663f614b-864a-4628-a976-924725dd2a5c"
+					(reference "#PWR030")
+					(unit 1)
+				)
+			)
 			(project "Template"
 				(path "/b7abe575-2b7a-4e47-9046-9769d7102f9d/c3e404eb-2e1f-4ab9-8da3-bc1a9ff0af28/5567a483-a138-4241-99fb-eb385b2c8ebc"
@@
 		)
 	)
+	(sheet_instances
+		(path "/"
+			(page "1")
+		)
+	)
