File: hardware/cba/kaman/Template.kicad_pcb (KiCad board)
At the start: 2 copper layers, 45 parts, among them J1 Conn_01x04_Pin, J2 Conn_01x04_Pin, J3 Barrel_Jack_MountingPin, J4 USB_C_Receptacle_USB2.0_16P, J5 Conn_01x02_Socket, Q1 MMDT5551, SW1 SW_Push, SW2 SW_Push, U1 ESP32-C6-MINI-1, U3 NEO-M8N, U4 AT24CS64-SSHM, U5 AZ1117-3.3, U6 CH340C, U7 PRTR5V0U2D

Commit message: hw(pcb): unrouted v0.1 pcb
Parts:
- C10, C11, C12, C5, D5, R8: moved to B.Cu
- moved R2 139.1 mm to (206.0, 75.1), turned to -90 degrees
- moved R1 134.7 mm to (202.2, 75.1), turned to 90 degrees
- moved C1 129.0 mm to (199.3, 73.6), turned to 90 degrees
- moved C2 128.6 mm to (199.3, 77.5), turned to -90 degrees
- moved JP2 126.4 mm to (205.5, 71.0), turned to -90 degrees
- moved JP1 122.4 mm to (202.8, 71.0), turned to -90 degrees
- moved U3 119.9 mm to (182.8, 91.0), turned to 90 degrees
- moved C4 119.4 mm to (181.4, 61.6), turned to 90 degrees
- moved SW2 116.8 mm to (195.4, 77.5)
- moved SW1 116.5 mm to (195.4, 73.6), turned to 180 degrees
- moved U1 116.3 mm to (190.0, 65.0)
- moved Q1 114.8 mm to (204.1, 75.1), turned to -90 degrees
- moved D6 111.6 mm to (215.1, 89.5), turned to -90 degrees
- moved C5 108.1 mm to (176.7, 80.1)
- moved J4 108.1 mm to (218.9, 65.4), turned to 90 degrees
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Routing:
- net +3.3V: vias 0 -> 1
- added copper zone on B.Cu, net GND
- added copper zone on F.Cu, net GND
Other:
- board outline added: 48.9 x 49 mm

Commit message: hw(pcb): unorganized overlay 0.1v pcb
Parts:
- removed C10: 100nF, Capacitor_SMD:C_0402_1005Metric_Pad0.74x0.62mm_HandSolder
- D5: footprint Diode_SMD:D_SOD-523 -> Diode_SMD:D_SOD-323
- moved C5 0.95 mm to (176.7, 81.0)
- moved R11 0.25 mm to (211.2, 63.5)
- moved R12 0.25 mm to (211.2, 67.5)
- moved U7 0.25 mm to (211.2, 65.5)
- moved U1 0.15 mm to (190.0, 64.8)
Connections:
- net Net-(J4-D+-PadA6) renamed /Project Architecture/IO Port/USB_P
- net Net-(J4-D--PadA7) renamed /Project Architecture/IO Port/USB_N
- net Net-(U6-UD+) renamed /Project Architecture/IO Port/USB2_N
- net Net-(U6-UD-) renamed /Project Architecture/IO Port/USB2_P
- J4 pad SH: (no net) -> GND
- U1 pad 12: unconnected-(U1-IO0-Pad12) -> GPS RX
- U1 pad 13: unconnected-(U1-IO1-Pad13) -> GPS TX
Routing:
- net +3.3V: track 0.00 -> 126.5 mm, vias 1 -> 3
- net EN: track 0.00 -> 29.2 mm, vias 0 -> 2
- net GPS TX: track 0.00 -> 22.3 mm
- net GPS RX: track 0.00 -> 21.8 mm, vias 0 -> 2
- net UART RX: track 0.00 -> 19.2 mm, vias 0 -> 2
- net GPIO 9: track 0.00 -> 14.0 mm
- net Net-(U3-SDA/~{SPI_CS}): track 0.00 -> 13.8 mm
- net UART TX: track 0.00 -> 13.5 mm
- net Net-(U3-SCL/SPI_CLK): track 0.00 -> 11.6 mm
- net Net-(D7-A): track 0.00 -> 10.7 mm
- net /Project Architecture/IO Port/USB2_P: track 0.00 -> 10.2 mm
- net SDA Oled: track 0.00 -> 9.37 mm
- net /Project Architecture/IO Port/USB2_N: track 0.00 -> 8.91 mm
- net SCL Oled: track 0.00 -> 8.63 mm
- net Net-(U3-V_BCKP): track 0.00 -> 7.74 mm, vias 0 -> 1
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- added copper zone on F.Cu, net +3.3V
- added copper zone on F.Cu, net VDD

Commit message: hw(pcb): final 0.2v pcb
Parts:
- removed AE1: Antenna, Connector_Coaxial:U.FL_Hirose_U.FL-R-SMT-1_Vertical
- added AE2: Antenna_Shield, Connector_Coaxial:SMA_Amphenol_132134-11_Vertical, F.Cu at (217.9, 103.1)
- added AE3: Antenna_Shield, Connector_Coaxial:U.FL_Hirose_U.FL-R-SMT-1_Vertical, F.Cu at (188.7, 105.7)
- added C10: 100nF, Capacitor_SMD:C_0603_1608Metric_Pad1.08x0.95mm_HandSolder, F.Cu at (215.2, 94.8)
- added C16: 10uF, Capacitor_SMD:C_0805_2012Metric_Pad1.18x1.45mm_HandSolder, F.Cu at (215.4, 96.7)
- added C17: 10uF, Capacitor_SMD:C_0805_2012Metric_Pad1.18x1.45mm_HandSolder, F.Cu at (205.4, 83.0)
- added C18: 10uF, Capacitor_SMD:C_0805_2012Metric_Pad1.18x1.45mm_HandSolder, F.Cu at (197.3, 80.5)
- added D10: LED, LED_SMD:LED_0603_1608Metric_Pad1.05x0.95mm_HandSolder, F.Cu at (188.1, 80.3)
- added D9: SD03C-MMD, Diode_SMD:D_SOD-323, F.Cu at (215.1, 93.0)
- added R14: 1K, Resistor_SMD:R_0603_1608Metric_Pad0.98x0.95mm_HandSolder, B.Cu at (201.3, 84.0)
- added R15: 6.8K, Resistor_SMD:R_0603_1608Metric_Pad0.98x0.95mm_HandSolder, B.Cu at (199.6, 84.0)
- added R16: 1K, Resistor_SMD:R_0603_1608Metric_Pad0.98x0.95mm_HandSolder, F.Cu at (188.1, 83.1)
- added SW3: SW_DIP_x01, Button_Switch_SMD:SW_DIP_SPSTx01_Slide_6.7x4.1mm_W8.61mm_P2.54mm_LowProfile, F.Cu at (198.3, 85.0)
- added U8: Ai-Thinker-Ra-01, RF_Module:Ai-Thinker-Ra-01-LoRa, F.Cu at (203.8, 96.6)
- added U9: SY6280AAAC, Package_TO_SOT_SMD:SOT-23-5, F.Cu at (201.0, 80.7)
- moved D8 11.8 mm to (205.4, 79.2), turned to -90 degrees
- moved C15 10.1 mm to (202.6, 78.0), turned to 180 degrees
- moved U5 6.27 mm to (209.1, 80.9), turned to 90 degrees
- moved J5 5.28 mm to (219.3, 91.7), turned to 180 degrees
- moved D6 5.13 mm to (218.6, 85.7), turned to 0 degrees
- moved C14 1.07 mm to (214.8, 86.3), turned to -90 degrees
- moved SW2 1.05 mm to (196.0, 76.6)
- moved SW1 1.05 mm to (196.0, 72.7)
- moved C2 1.05 mm to (199.8, 76.6)
- moved C1 1.05 mm to (199.8, 72.7)
- moved R5 0.90 mm to (175.8, 73.2)
- moved R6 0.90 mm to (175.8, 75.0)
- moved J2 0.88 mm to (179.5, 74.2)
- moved JP2 0.20 mm to (205.3, 71.0)
- moved J4 0.15 mm to (218.8, 65.4)
Connections:
- C15 pad 1: +3.3V -> Net-(D8-A2)
- D8 pad 2: +3.3V -> Net-(D8-A2)
- U1 pad 15: unconnected-(U1-IO6-Pad15) -> NSS LoRa
- U1 pad 16: unconnected-(U1-IO7-Pad16) -> MISO LoRa
- U1 pad 19: unconnected-(U1-IO14-Pad19) -> MOSI LoRa
- U1 pad 20: unconnected-(U1-IO15-Pad20) -> SCK LoRa
- U1 pad 22: unconnected-(U1-IO8-Pad22) -> BUSY LoRa
- U1 pad 24: unconnected-(U1-IO18-Pad24) -> DIO1 LoRa
- U5 pad 2: +3.3V -> Net-(D8-A2)
- U6 pad 5: /Project Architecture/IO Port/USB2_N -> /Project Architecture/IO Port/USB2_P
- U6 pad 6: /Project Architecture/IO Port/USB2_P -> /Project Architecture/IO Port/USB2_N
- U7 pad 1: /Project Architecture/IO Port/USB2_N -> /Project Architecture/IO Port/USB2_P
- U7 pad 3: /Project Architecture/IO Port/USB2_P -> /Project Architecture/IO Port/USB2_N
- U7 pad 4: /Project Architecture/IO Port/USB_P -> /Project Architecture/IO Port/USB_N
- U7 pad 6: /Project Architecture/IO Port/USB_N -> /Project Architecture/IO Port/USB_P
Routing:
- net BUSY LoRa: track 0.00 -> 36.2 mm, vias 0 -> 2
- net NSS LoRa: track 0.00 -> 35.5 mm
- net DIO1 LoRa: track 0.00 -> 34.1 mm, vias 0 -> 2
- net MISO LoRa: track 0.00 -> 33.2 mm
- net MOSI LoRa: track 0.00 -> 30.2 mm
- net SCK LoRa: track 0.00 -> 27.8 mm
- net Net-(U9-EN): track 0.00 -> 10.9 mm, vias 0 -> 2
- net +3.3V: track 126.5 -> 134.4 mm, vias 3 -> 8
- net Net-(AE2-A): track 0.00 -> 6.29 mm
- net Net-(D8-A2): track 0.00 -> 5.24 mm, vias 0 -> 2
- net GND: track 4.14 -> 9.08 mm, vias 225 -> 110
- net Net-(U9-ISET): track 0.00 -> 3.17 mm, vias 0 -> 1
- net VDD: track 3.15 -> 0.00 mm
- net Net-(D10-K): track 0.00 -> 2.77 mm
- net /Project Architecture/IO Port/USB_P: track 3.28 -> 5.88 mm
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- added copper zone on F.Cu, net Net-(D8-A2)
Other:
- board text added: "3.3V"
